File: camera-Power_supply/ezs-camera.sch (KiCad schematic (older format))
At the start: 42 parts, among them J1 CONN_01X12, J2 CONN_02X12, J3 STEP, J4 POWER, J5 BAT, J6 PWR_LED, U1 ULN2003, U2 BQ2407x, U3 LM3405, U4 TPS6123x

Commit message: first
Parts:
- J1: symbol CONN_01X12 -> Conn_01x12
- J3: symbol CONN_01X05 -> Conn_01x05
Changed lines of the file:
@@
 LIBS:tps6123x
 LIBS:symbols
+LIBS:_saved_ezs-camera-rescue
 LIBS:ezs-camera-cache
+LIBS:lm3405
 EELAYER 26 0
 EELAYER END
@@
 $EndDescr
 $Comp
-L CONN_01X12 J1
+L Conn_01x12 J1
 U 1 1 597E7495
 P 8050 1750
@@
 $EndComp
 $Comp
-L CONN_01X05 J3
+L Conn_01x05 J3
 U 1 1 597E80E3
 P 8600 3750
