File: camera-Power_supply/ezs-camera.kicad_pcb (KiCad board)
At the start: 2 copper layers, 47 x 51 mm, 42 parts, among them J1 CONN_01X12, J2 CONN_02X12, J3 STEP, J4 POWER, J5 BAT, J6 PWR_LED, U1 ULN2003, U2 BQ2407x, U3 LM3405, U4 TPS6123x

Commit message: v1.0 prvni prototyp odeslany vyrobit
Parts:
- removed J4: POWER, Wire_Connections_Bridges:WireConnection_2.50mmDrill
- J3, J5, J6: moved to F.Cu
- moved J6 40.4 mm to (134.6, 152.9), turned to 270 degrees
- moved J3 32.6 mm to (127.5, 154.9), turned to 180 degrees
- moved C5 27.5 mm to (130.4, 137.7), turned to 0 degrees
- moved U1 26.6 mm to (124.3, 146.1), turned to 270 degrees
- moved C4 24.8 mm to (130.3, 135.6), turned to 0 degrees
- moved L1 23.2 mm to (128.4, 130.1), turned to 270 degrees
- moved R7 21.2 mm to (136.5, 138.0), turned to 0 degrees
- moved C8 20.2 mm to (150.4, 146.1), turned to 0 degrees
- moved R1 19.3 mm to (146.1, 150.4)
- moved U2 18.0 mm to (147.2, 141.9)
- moved R3 18.0 mm to (144.2, 138.6)
- moved C12 18.0 mm to (146.5, 136.6)
- moved C2 18.0 mm to (143.9, 142.2)
- moved D3 18.0 mm to (152.8, 142.2)
- moved R5 18.0 mm to (152.8, 138.4)
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Connections:
- J1 pad 12: Net-(J1-Pad12) -> GND
Routing:
- net +5V: track 47.4 -> 123.7 mm
- net Net-(C4-Pad1): track 0.00 -> 26.1 mm
- net +4,4V: track 12.7 -> 35.7 mm
- net /PGOOD: track 19.0 -> 37.8 mm
- net /LED_EN: track 1.95 -> 18.5 mm
- net +5P: track 0.35 -> 14.7 mm, vias 0 -> 1
- net Net-(C5-Pad2): track 16.1 -> 28.8 mm
- net Net-(J2-Pad13): track 12.5 -> 0.00 mm
- net Net-(J2-Pad11): track 11.8 -> 0.00 mm
- net Net-(C3-Pad2): track 0.00 -> 9.96 mm
- net /BAT: track 0.27 -> 9.47 mm
- net Net-(J2-Pad21): track 0.00 -> 8.09 mm
- net Net-(J5-Pad1): track 14.5 -> 6.64 mm
- net Net-(J3-Pad1): track 0.00 -> 7.68 mm
- net Net-(J2-Pad19): track 17.6 -> 11.2 mm
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- added copper zone on F.Cu, net +5P
- added copper zone on F.Cu, net /BAT
- removed copper zone on F.Cu, net /BATT
- removed copper zone on F.Cu, net Net-(C3-Pad2)
- removed copper zone on F.Cu, net Net-(C4-Pad1)
Other:
- net class Default: clearance 0.1 -> 0.1524
- rule trace_clearance: 0.1 -> 0.1524
- rule via_min_drill: 0.3 -> 0.4
- board text added: "+5V"
- board text added: "GND"
