File: camera-Power_supply/_autosave-ezs-camera.kicad_pcb (KiCad board)
At the start: 2 copper layers, 47 x 51 mm, 42 parts, among them J1 CONN_01X12, J2 CONN_02X12, J3 STEP, J4 POWER, J5 BAT, J6 PWR_LED, U1 ULN2003, U2 BQ2407x, U3 LM3405, U4 TPS6123x

Commit message: v1.1 redesign
Connections:
- J1 pad 1: (no net) -> Net-(J1-Pad1)
- J1 pad 10: (no net) -> Net-(J1-Pad10)
- J1 pad 11: (no net) -> Net-(J1-Pad11)
- J1 pad 12: GND -> Net-(J1-Pad12)
- J1 pad 2: (no net) -> Net-(J1-Pad2)
- J1 pad 3: (no net) -> Net-(J1-Pad3)
- J1 pad 4: (no net) -> Net-(J1-Pad4)
- J1 pad 5: (no net) -> Net-(J1-Pad5)
- J1 pad 6: (no net) -> Net-(J1-Pad6)
- J1 pad 7: (no net) -> Net-(J1-Pad7)
- J1 pad 8: (no net) -> Net-(J1-Pad8)
- J1 pad 9: (no net) -> Net-(J1-Pad9)
- J2 pad 1: (no net) -> Net-(J2-Pad1)
- J2 pad 10: (no net) -> Net-(J2-Pad10)
- J2 pad 12: (no net) -> Net-(J2-Pad12)
- J2 pad 16: (no net) -> Net-(J2-Pad16)
- J2 pad 17: (no net) -> Net-(J2-Pad17)
- J2 pad 18: (no net) -> Net-(J2-Pad18)
- J2 pad 22: (no net) -> Net-(J2-Pad22)
- J2 pad 24: (no net) -> Net-(J2-Pad24)
- J2 pad 3: (no net) -> Net-(J2-Pad3)
- J2 pad 5: (no net) -> Net-(J2-Pad5)
- J2 pad 7: (no net) -> Net-(J2-Pad7)
- J2 pad 8: (no net) -> Net-(J2-Pad8)
- U1 pad 10: (no net) -> Net-(U1-Pad10)
- U1 pad 11: (no net) -> Net-(U1-Pad11)
- U1 pad 12: (no net) -> Net-(U1-Pad12)
- U1 pad 5: (no net) -> Net-(U1-Pad5)
- U1 pad 6: (no net) -> Net-(U1-Pad6)
- U1 pad 7: (no net) -> Net-(U1-Pad7)
